File: Expansion_Card_Retrofit.kicad_sch (KiCad schematic)
At the start: 54 parts, among them P1 USB_C_Plug_USB2.0, U1 RP2350_60QFN, U2 CCGM1A1, U4 W25X20CLUXIG-TR, U5 W25X20CLUXIG-TR, U6 NCP163AFCT330T2G, Y1 S3A2505-100.000-L-X1-R, Y2 ABM8-272-T3

Commit message: update
Parts:
- removed D5, D6, D7, D8: 16-213SDRC/S530-A3/TR8, LED_SMD:LED_0402_1005Metric, symbol Device:LED
- removed R10, R11, R9: 60R4, Resistor_SMD:R_0201_0603Metric, symbol Device:R_US
- removed U6: NCP163AFCT330T2G, Package_CSP:WLCSP-4_0.64x0.64mm_P0.35mm, symbol Regulator_Linear:NCP163AFCT330T2G
- added C10, C100, C101, C102, C103, C104, C105, C106, C12, C17, C22, C27, C34, C39, C42, C47, C50, C52, C55, C58, C66, C73, C78, C89, C9, C99: 100n, Capacitor_SMD:C_0402_1005Metric, symbol Device:C
- added C107, C108, C109, C110, C13, C18, C21, C26, C35, C40, C41, C51, C54, C57, C65, C74, C79, C81, C90: 1u, Capacitor_SMD:C_0402_1005Metric, symbol Device:C
- added C11, C111, C112, C113, C114, C115, C116, C117, C16, C19, C20, C23, C24, C25, C28, C29, C30, C31, C32, C33, C36, C37, C38, C43, C44, C45, C46, C49, C53, C56, C59, C60, C61, C62, C63, C64, C67, C68, C69, C70, C71, C72, C75, C76, C77, C80, C82, C91, C92, C93, C94, C95, C96, C97, C98: 10n, Capacitor_SMD:C_0201_0603Metric, symbol Device:C
- added D12, D13: PTVS5V0Z1USK, Diode_SMD:Nexperia_DSN1608-2_1.6x0.8mm, symbol Diode:PTVS5V0Z1USK
- added JP1: Jumper_2_Open, Jumper:SolderJumper-2_P1.3mm_Open_RoundedPad1.0x1.5mm, symbol Jumper:Jumper_2_Open
- added R21, R25, R28: 200R, Resistor_SMD:R_0201_0603Metric, symbol Device:R_US
- added R22, R31: 100R, Resistor_SMD:R_0201_0603Metric, symbol Device:R_US
- added R23: 5K1, Resistor_SMD:R_0201_0603Metric, symbol Device:R_US
- added R26, R27, R29, R30, R32, R33, R34: 0R, Resistor_SMD:R_0201_0603Metric, symbol Device:R_US
- added TH1: PTSLR06038V075, Capacitor_SMD:C_0603_1608Metric, symbol Device:Thermistor_PTC_US
- added U3: TVS0500DRV, Package_SON:WSON-6-1EP_2x2mm_P0.65mm_EP1x1.6mm, symbol Power_Protection:TVS0500DRV
- C1, C2, C3: footprint Capacitor_SMD:C_0201_0603Metric -> Capacitor_SMD:C_0402_1005Metric
- C4, C5, C6: footprint (none) -> Capacitor_SMD:C_0402_1005Metric; MPN (none) -> GRM155C61E475ME15D
- C7, C8: value 100n -> 15p; footprint Capacitor_SMD:C_0201_0603Metric -> Capacitor_SMD:C_0402_1005Metric
- D1, D10, D11, D2, D3, D4: MPN (none) -> 16-213SDRC/S530-A3/TR8
- D9: MPN (none) -> DT1240A-08LP3810
- P1: value USB_C_Plug_USB2.0 -> 1054440011
- R1, R17, R18, R19, R2, R20, R4: footprint (none) -> Resistor_SMD:R_0201_0603Metric
- R12: value 60R4 -> 5K1; now not fitted; now left out of the parts list
- R15: value 30R1 -> 5K1
- R16: value 30R1 -> 0R; now not fitted; now left out of the parts list
- R3: footprint (none) -> Resistor_SMD:R_0402_1005Metric
- TP5, TP6: footprint (none) -> TestPoint:TestPoint_Pad_D1.0mm
- U1: MPN (none) -> RP2350A
- U2: MPN (none) -> CCGM1A1-BGA324
- U4, U5: value W25X20CLUXIG-TR -> W25Q32RVXHJQ TR; MPN (none) -> W25Q32RVXHJQ TR
- Y1: footprint S3A2505-100.000-L-X1-R:OSC_S3A2505-100.000-L-X1-R -> ProjectLibrary:OSC_S3A2505-100.000-L-X1-R; MPN (none) -> S3A2505-100.000-L-X1-R
- Y2: MPN (none) -> ABM8-272-T3
Connections:
- net +0V9 is gone; now on net +1V: U2.F9 (VDD), U2.G10 (VDD), U2.G12 (VDD), U2.G6 (VDD), U2.G8 (VDD), U2.H11 (VDD), U2.H13 (VDD), U2.H7 (VDD), U2.H9 (VDD), U2.J10 (VDD), U2.J12 (VDD), U2.J6 (VDD), U2.J8 (VDD), U2.K11 (VDD), U2.K13 (VDD), U2.K7 (VDD), U2.K9 (VDD), U2.L10 (VDD), U2.L12 (VDD), U2.L6 (VDD), U2.L8 (VDD), U2.M11 (VDD), U2.M13 (VDD), U2.M7 (VDD), U2.M9 (VDD), U2.N10 (VDD), U2.N6 (VDD), U2.N8 (VDD), U2.P16 (VDD_PLL), U2.T16 (VDD_SER_PLL), U2.U12 (VDD_SER), U2.V17 (VDD_SER)
- net K7 is gone; now on an unnamed net: R12.2
- net +1V1: now also C54.1, C55.1, C56.1
- net +2V5: now also R12.1, R15.1, C11.1, C12.1, C13.1, C16.1, C17.1, C18.1, C19.1, C20.1, C21.1, C22.1, C23.1, C24.1, C25.1, C26.1, C27.1, C28.1, C29.1, C30.1, C31.1, C32.1, C33.1, C34.1, C35.1, C36.1, C37.1, C38.1, C39.1, C40.1, C41.1, C42.1, C43.1, C44.1, C45.1, C46.1, C47.1, C49.1, C50.1, C51.1, C57.1, C58.1, C59.1, C60.1, C61.1, C62.1, C65.1, C66.1, C67.1, C68.1, C69.1, C70.1, C71.1, C72.1, C73.1, C74.1, C75.1, C76.1, C77.1, C78.1, C79.1, R26.1, R27.1, R31.1, R34.1; no longer U2.N18 (VDD_SB), U2.T14 (VDD_CLK), U2.T18 (VDD_SB), Y1.1 (ENABLE/DISABLE)
- net +3V3: now also R3.2, C80.1, C81.1
- net GND: now also U2.U14 (GND/SER_RX1_P), U2.V14 (GND/SER_RX1_N), C100.2, C101.2, C102.2, C103.2, C104.2, C105.2, C106.2, C107.2, C108.2, C109.2, C11.2, C110.2, C111.2, C112.2, C113.2, C114.2, C115.2, C116.2, C117.2, C12.2, C13.2, C16.2, C17.2, C18.2, C19.2, C20.2, C21.2, C22.2, C23.2, C24.2, C25.2, C26.2, C27.2, C28.2, C29.2, C30.2, C31.2, C32.2, C33.2, C34.2, C35.2, C36.2, C37.2, C38.2, C39.2, C40.2, C41.2, C42.2, C43.2, C44.2, C45.2, C46.2, C47.2, C49.2, C50.2, C51.2, C52.2, C53.2, C54.2, C55.2, C56.2, C57.2, C58.2, C59.2, C60.2, C61.2, C62.2, C63.2, C64.2, C65.2, C66.2, C67.2, C68.2, C69.2, C70.2, C71.2, C72.2, C73.2, C74.2, C75.2, C76.2, C77.2, C78.2, C79.2, C80.2, C81.2, C82.2, C89.2, C90.2, C91.2, C92.2, C93.2, C94.2, C95.2, C96.2, C97.2, C98.2, C99.2, D12.2 (A), D13.2 (A), JP1.1 (A), R21.2, R22.2, R23.2, R25.1, R28.1, R29.2, R30.2, U3.1 (GND), U3.2 (GND), U3.3 (GND), U3.7 (GND); no longer U2.U14 (GND), U2.U16 (GND), U2.V14 (GND), U2.V16 (GND)
- net LED2: now also R6.1; no longer R7.1
- net LED4: now also R7.1
- net LED5: now also R8.1
- net USB_DN: now also D13.1 (K); no longer D9.8 (K7)
- net USB_DP: now also D12.1 (K); no longer D9.2 (K2)
- net VBUS: now also TH1.1, U3.4 (IN), U3.5 (IN), U3.6 (IN); no longer D9.4 (K3), P1.A4 (VBUS), P1.A9 (VBUS), P1.B4 (VBUS), P1.B9 (VBUS)
- net RX2_N: now reaches P1.A10 (RX2-)
- net RX2_N: now also D9.4 (K3), R32.1
- net RX2_P: now reaches P1.A11 (RX2+)
- net RX2_P: now also D9.7 (K6), R33.1
- net at P1.A5 (CC), R1.1: no longer D9.7 (K6)
- net TX2_P: now reaches P1.B2 (TX2+)
- net TX2_P: now also D9.6 (K5), C9.1
- net TX2_N: now reaches P1.B3 (TX2-)
- net TX2_N: now also D9.5 (K4), C10.1
- net at U2.N16 (NC/VDD_SER): now also R16.2
- net CC_CFG_CTRL_EN: now reaches U2.B1 (IO_WC_A8)
- net CC_CFG_CTRL_EN: now also U1.36 (GPIO24), R23.1; no longer U1.33 (GPIO21)
- net CC_CFG_CTRL_CLK: now reaches U1.32 (GPIO20), U2.B2 (IO_WC_B8)
- net at U2.D1 (IO_WC_A5): no longer U1.35 (GPIO23)
- net CC_CFG_CTRL_VALID: now reaches U1.34 (GPIO22), U2.D2 (IO_WC_B5)
- net POR_EN: now reaches U2.U1 (POR_EN/IO_WA_A3)
- net POR_EN: now also R34.2
- net at U1.60 (QSPI_SS), U4.1 (~{CS}): now also JP1.2 (B)
- net SER_CLK_P: now reaches Y1.4 (CLK+)
- net SER_CLK_P: now also U2.T12 (SER_CLK); no longer R15.1
- net +1V: now reaches R16.1
- net +1V: now also U2.T14 (VDD_CLK), C100.1, C101.1, C102.1, C103.1, C104.1, C105.1, C106.1, C107.1, C108.1, C109.1, C110.1, C111.1, C112.1, C113.1, C114.1, C115.1, C116.1, C117.1, C53.1, C63.1, C64.1, C82.1, C89.1, C90.1, C91.1, C92.1, C93.1, C94.1, C95.1, C96.1, C97.1, C98.1, C99.1; no longer Y1.5 (CLK-)
- net SER_CLK_N: now reaches U2.T13 (SER_CLK_N)
- net SER_CLK_N: now also Y1.5 (CLK-); no longer R16.2
- net GPIO23_GPOUT1: now reaches U2.P12 (CLK1/IO_SB_A7)
- net GPIO23_GPOUT1: now also U1.35 (GPIO23)
- net GPIO21_GPOUT0: now reaches U2.P14 (CLK2/IO_SB_A6)
- net GPIO21_GPOUT0: now also U1.33 (GPIO21)
- net C_TX2_N: now reaches U2.R17 (IO_SB_A1/SER_TX2_P)
- net C_TX2_N: now also C9.2
- net C_TX2_P: now reaches U2.R18 (IO_SB_B1/SER_TX2_N)
- net C_TX2_P: now also C10.2
- net R_TX2_N: now reaches U2.U17 (IO_SB_A0/SER_RX2_P)
- net R_TX2_N: now also R33.2
- net R_TX2_P: now reaches U2.U18 (IO_SB_B0/SER_RX2_N)
- net R_TX2_P: now also R32.2
- net at U2.V12 (SER_RTERM): now also R21.1
- net power_supply/PG: now reaches U2.K18 (IO_EA_A2)
- net at R15.2: now also Y1.1 (ENABLE/DISABLE); no longer U2.T12 (SER_CLK)
- net at U2.V15 (POR_ADJ): now also C52.1, R22.1, R31.2
- net C_TX_N renamed C_TX1_N
- net C_TX_P renamed C_TX1_P
- net LED1: no longer names the net of U2.B3 (IO_NA_B0)
- net LED1: no longer R6.1
- net LED3: no longer names the net of U2.B4 (IO_NA_B1)
- net LED3: no longer R8.1
- net LED6: no longer names the net of U2.B6 (IO_NA_B4)
- net LED7: no longer names the net of U2.A8 (IO_NA_A7)
- net LED7: no longer R12.1
- net RX_N renamed RX1_N
- net RX_P renamed RX1_P
- net TX_N renamed TX1_N
- net TX1_N: now also D9.2 (K2); no longer D9.6 (K5)
- net TX_P renamed TX1_P
- net TX1_P: now also D9.8 (K7); no longer D9.5 (K4)
- new net: P1.A4 (VBUS), P1.A9 (VBUS), P1.B4 (VBUS), P1.B9 (VBUS), TH1.2
- new net: R30.1, U2.U16 (GND/SER_TX1_P)
- new net: R27.2, R28.2, U2.N18 (VDD_SB/SER_TERM3)
- new net: R25.2, R26.2, U2.T18 (VDD_SB/SER_TERM3)
- new net: R29.1, U2.V16 (GND/SER_TX1_N)
- no-connect marks 6 -> 130
Other:
- added sheet power_supply (POWER.kicad_sch)
- note added: "1V 2V5 3V3"
- note added: "5V"
- note added: "CX1 = 2(CL - Cstray) CL = 10pF Cstray = 2pF CX1 = 2(10-2) = 16pF"
- note added: "FPGA DECOUPLING 100MHZ"
- note added: "TODO: ADD CORE DECOUPLING"
- note added: "VDD_PLL"
- note added: "VDD_SER"
- note added: "VDD_SER_PLL"
- note added: "x24"
- note removed: "TODO: ADD APPROPRIATE TERMINAISON"
- note removed: "TODO: change cap value"
- moved on the sheet: C1, C2, C3, C4, C5, C6, C7, D1, D10, D11, D2, D3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

Commit message: first routing
Parts:
- removed C49: 10n, Capacitor_SMD:C_0201_0603Metric, symbol Device:C
- removed C50: 100n, Capacitor_SMD:C_0402_1005Metric, symbol Device:C
- removed C51: 1u, Capacitor_SMD:C_0402_1005Metric, symbol Device:C
- removed JP1: Jumper_2_Open, Jumper:SolderJumper-2_P1.3mm_Open_RoundedPad1.0x1.5mm, symbol Jumper:Jumper_2_Open
- removed R18, R19, R20: 5K1, Resistor_SMD:R_0201_0603Metric, symbol Device:R_US
- removed U5: W25Q32RVXHJQ TR, Package_SON:Winbond_USON-8-1EP_3x2mm_P0.5mm_EP0.2x1.6mm, symbol Memory_Flash:MX25R3235FZNxx0
- added D14, D15, D16: PTVS5V0Z1USK, Diode_SMD:Nexperia_DSN1608-2_1.6x0.8mm, symbol Diode:PTVS5V0Z1USK
- added D5, D6: 16-213SDRC/S530-A3/TR8, LED_SMD:LED_0402_1005Metric, symbol Device:LED
- added J1, J4: Conn_02x02_Odd_Even, Connector_PinHeader_1.00mm:PinHeader_2x02_P1.00mm_Horizontal, symbol Connector_Generic:Conn_02x02_Odd_Even
- added J3: 5024302030, Connector_Molex:Molex_SlimStack_502430-2010_2x10_P0.40mm_Vertical, symbol Connector_Generic:Conn_02x10_Odd_Even
- added R36, R37: 60R4, Resistor_SMD:R_0201_0603Metric, symbol Device:R_US
- added R38, R39: 0R, Resistor_SMD:R_0201_0603Metric, symbol Device:R_US
Connections:
- net +2V5: now also D14.1 (K), D5.2 (A), D6.2 (A), J3.1 (Pin_1), J4.2 (Pin_2), R38.1, R39.1
- net GND: now also D14.2 (A), D15.2 (A), D16.2 (A), J1.3 (Pin_3), J1.4 (Pin_4), J3.10 (Pin_10), J3.12 (Pin_12), J3.14 (Pin_14), J3.16 (Pin_16), J3.18 (Pin_18), J3.19 (Pin_19), J3.2 (Pin_2), J3.20 (Pin_20), J3.4 (Pin_4), J3.6 (Pin_6), J3.8 (Pin_8), J4.4 (Pin_4); no longer U2.U4 (CFG_MD2/IO_WA_A1), U2.V4 (CFG_MD3/IO_WA_B1)
- net LED0: now also U2.A8 (IO_NA_A7); no longer U2.A3 (IO_NA_A0)
- net LED2: now also R7.1, U2.A12 (IO_NB_B4); no longer R6.1, U2.A4 (IO_NA_A1)
- net LED4: now also U2.A14 (IO_NB_B7), R36.1; no longer R7.1, U2.B5 (IO_NA_A2)
- net LED5: now also U2.B14 (IO_NB_A7), R37.1; no longer R8.1, U2.A6 (IO_NA_A4)
- net RUN: now also J1.1 (Pin_1)
- net RX0: now also U2.C18 (IO_EB_A4); no longer U2.M4 (IO_WB_B1)
- net RX1: now also U2.C17 (IO_EB_B4); no longer U2.L4 (IO_WB_B2)
- net TX0: now also U2.D18 (IO_EB_A2); no longer U2.M3 (IO_WB_A1)
- net TX1: now also U2.D17 (IO_EB_B2); no longer U2.L3 (IO_WB_A2)
- net LED1: now reaches U2.A9 (IO_NB_B0)
- net LED1: now also R6.1
- net LED3: now reaches U2.B12 (IO_NB_A4)
- net LED3: now also R8.1
- net at U2.N3 (IO_WA_A8/~{SPI_CS}): now also J3.11 (Pin_11)
- net at U2.P1 (IO_WA_A7/SPI_D1): now also J3.5 (Pin_5)
- net at U2.R2 (IO_WA_B6/SPI_D2): now also J3.7 (Pin_7)
- net at U2.P2 (IO_WA_B7/SPI_D0): now also J3.3 (Pin_3)
- net at U2.N4 (IO_WA_B8/SPI_CLK): now also J3.13 (Pin_13)
- net at U2.R1 (IO_WA_A6/SPI_D3): now also J3.9 (Pin_9)
- net IO_P: now reaches U2.E3 (IO_WC_A4)
- net IO_P: now also D16.1 (K), J4.1 (Pin_1)
- net IO_N: now reaches U2.E4 (IO_WC_B4)
- net IO_N: now also D15.1 (K), J4.3 (Pin_3)
- net ~{FLASH_CS}: now reaches R12.2, U1.60 (QSPI_SS), U4.1 (~{CS})
- net ~{FLASH_CS}: now also J1.2 (Pin_2)
- net FLASH_S1: now reaches U1.59 (QSPI_SD1), U4.2 (SO/SIO1)
- net FLASH_S2: now reaches U1.58 (QSPI_SD2), U4.3 (~{WP}/SIO2)
- net FLASH_S0: now reaches U1.57 (QSPI_SD0), U4.5 (SI/SIO0)
- net FLASH_CLK: now reaches U1.56 (QSPI_SCLK), U4.6 (SCLK)
- net FLASH_S3: now reaches U1.55 (QSPI_SD3), U4.7 (~{RESET}/SIO3)
- net GPIO21_GPOUT0: no longer names the net of U1.33 (GPIO21)
- net GPIO21_GPOUT0: no longer U2.P14 (CLK2/IO_SB_A6)
- new net CFG_MD2/IO_WA_A1: J3.15 (Pin_15), R38.2, U2.U4 (CFG_MD2/IO_WA_A1)
- new net CFG_MD3/IO_WA_B1: J3.17 (Pin_17), R39.2, U2.V4 (CFG_MD3/IO_WA_B1)
- new net K4: D5.1 (K), R36.2
- new net K5: D6.1 (K), R37.2
- no-connect marks 130 -> 124
Other:
- moved on the sheet: C10, C16, C17, C18, C19, C20, C21, C22, C23, C24, C25, C26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

Commit message: Layout and add sensor
Parts:
- removed D12, D13, D14: PTVS5V0Z1USK, Diode_SMD:Nexperia_DSN1608-2_1.6x0.8mm, symbol Diode:PTVS5V0Z1USK
- added JP1: Jumper_2_Small_Open, Jumper:SolderJumper-2_P1.3mm_Open_RoundedPad1.0x1.5mm, symbol Jumper:Jumper_2_Small_Open
- added MK1: CMM-4737DT-26386-TR, Sensor_Audio:ST_HLGA-6_3.76x4.72mm_P1.65mm, symbol Sensor_Audio:MP45DT02
- added R18, R19, R20: 5K1, Resistor_SMD:R_0201_0603Metric, symbol Device:R_US
- added U10: TMP110D, Package_SON:Texas_X2SON-5_0.8x0.8mm_P0.48mm, symbol Sensor_Temperature:TMP110D
- added U5: USB3740B-AI2, Package_DFN_QFN:UQFN-10_1.3x1.8mm_P0.4mm, symbol Interface_USB:USB3740B-AI2
- added U9: ISM330DHCX, Package_LGA:LGA-14_3x2.5mm_P0.5mm_LayoutBorder3x4y, symbol Sensor_Motion:ISM330DHCX
- U4: value W25Q32RVXHJQ TR -> W25Q16JLUXIG TR
Connections:
- net +2V5: now also JP1.2 (B), R18.1, R19.1, R20.1, U10.5 (V+), U9.1 (SDO/SA0), U9.12 (CS), U9.5 (VDDIO), U9.8 (VDD); no longer J4.2 (Pin_2)
- net GND: now also J4.2 (Pin_2), MK1.1 (GND), MK1.3 (GND), U10.1 (GND), U10.3 (ADD0), U5.3 (OE_N), U5.8 (GND), U9.6 (GND), U9.7 (GND)
- net HSTX_0_N: now also U2.L2 (IO_WB_B3); no longer U2.N2 (IO_WB_B0)
- net HSTX_0_P: now also U2.L1 (IO_WB_A3); no longer U2.N1 (IO_WB_A0)
- net HSTX_1_N: now also U2.H2 (IO_WB_B7); no longer U2.L2 (IO_WB_B3)
- net HSTX_1_P: now also U2.H1 (IO_WB_A7); no longer U2.L1 (IO_WB_A3)
- net HSTX_3_N: now also U2.N2 (IO_WB_B0); no longer U2.H2 (IO_WB_B7)
- net HSTX_3_P: now also U2.N1 (IO_WB_A0); no longer U2.H1 (IO_WB_A7)
- net USB_DN: now also U5.7 (DM_2); no longer P1.A6 (D+)
- net USB_DP: now also U5.6 (DP_2); no longer P1.A7 (D-)
- net VBUS: now also U5.5 (VDD)
- net IMU_INT2: now reaches U2.B8 (IO_NA_B7)
- net IMU_INT2: now also U9.9 (INT2)
- net IMU_INT1: now reaches U2.C5 (IO_NA_B2)
- net IMU_INT1: now also U9.4 (INT1)
- net SDA0: now reaches U2.C6 (IO_NA_A3)
- net SDA0: now also R19.2, U10.4 (SDA), U9.14 (SDA)
- net SCL0: now reaches U2.D6 (IO_NA_B3)
- net SCL0: now also R20.2, U10.2 (SCL), U9.13 (SCL)
- net D_EN: now reaches U2.V7 (IO_SA_B3)
- net D_EN: now also R18.2, U5.4 (S)
- net MIC_CLK: now reaches U2.F18 (IO_EB_A0)
- net MIC_CLK: now also MK1.4 (CLK)
- net MIC_LR: now reaches U2.G17 (IO_EA_B7)
- net MIC_LR: now also MK1.2 (LR)
- net MIC_DOUT: now reaches U2.G18 (IO_EA_A7)
- net MIC_DOUT: now also MK1.5 (DOUT)
- net K5 renamed K8
- new net: JP1.1 (A), MK1.6 (VDD)
- new net C_USB_DN: P1.A7 (D-), U5.9 (DM)
- new net C_USB_DP: P1.A6 (D+), U5.10 (DP)
Other:
- note removed: "TODO: ADD CORE DECOUPLING"
- title: Expansion Card Template -> Expansion Card FPGA Accelerator
- moved on the sheet: C16, C17, C18, C19, C2, C20, C21, C22, C23, C24, C25, C26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

Commit message: update on layout first drc done
Parts:
- removed C4, C5: 4u7, Capacitor_SMD:C_0402_1005Metric, symbol Device:C
- removed L1: 3u3, RP2350_60QFN_minimal:L_pol_2016, symbol Device:L
- added FID1, FID2, FID3, FID4, FID5, FID6: Fiducial, Fiducial:Fiducial_0.5mm_Mask1mm, symbol Mechanical:Fiducial
- added N1: Housing, ProjectLibrary:Enclosure, symbol Mechanical:Housing
- added R41, R42, R43, R44: 5K1, Resistor_SMD:R_0201_0603Metric, symbol Device:R_US
- added U11: MMC5633NJL, Package_BGA:WLP-4_0.86x0.86mm_P0.4mm, symbol Sensor_Magnetic:MMC5633NJL
- U1: value RP2350_60QFN -> RP2350A
Connections:
- net +1V is gone; now on net +1V1: C100.1, C101.1, C102.1, C103.1, C104.1, C105.1, C106.1, C107.1, C108.1, C109.1, C110.1, C111.1, C112.1, C113.1, C114.1, C115.1, C116.1, C117.1, C53.1, C63.1, C64.1, C82.1, C89.1, C90.1, C91.1, C92.1, C93.1, C94.1, C95.1, C96.1, C97.1, C98.1, C99.1, R16.1, U2.F9 (VDD), U2.G10 (VDD), U2.G12 (VDD), U2.G6 (VDD), U2.G8 (VDD), U2.H11 (VDD), U2.H13 (VDD), U2.H7 (VDD), U2.H9 (VDD), U2.J10 (VDD), U2.J12 (VDD), U2.J6 (VDD), U2.J8 (VDD), U2.K11 (VDD), U2.K13 (VDD), U2.K7 (VDD), U2.K9 (VDD), U2.L10 (VDD), U2.L12 (VDD), U2.L6 (VDD), U2.L8 (VDD), U2.M11 (VDD), U2.M13 (VDD), U2.M7 (VDD), U2.M9 (VDD), U2.N10 (VDD), U2.N6 (VDD), U2.N8 (VDD), U2.P16 (VDD_PLL), U2.T14 (VDD_CLK), U2.T16 (VDD_SER_PLL), U2.U12 (VDD_SER), U2.V17 (VDD_SER)
- net +2V5: now also MK1.6 (VDD), R41.1, R42.1, R43.1, R44.1, U11.B1 (VDD); no longer JP1.2 (B)
- net +3V3: now also U1.49 (VREG_VIN), U5.5 (VDD)
- net GND: now also U11.A1 (VSA)
- net MIC_DOUT: now also JP1.2 (B); no longer MK1.5 (DOUT)
- net SCL0: no longer U10.2 (SCL)
- net SDA0: no longer U10.4 (SDA)
- net VBUS: no longer U1.49 (VREG_VIN), U5.5 (VDD)
- net SDA2: now reaches U2.C13 (IO_NB_B6)
- net SDA2: now also U10.4 (SDA), R43.2
- net SCL2: now reaches U2.C14 (IO_NB_B8)
- net SCL2: now also U10.2 (SCL), R44.2
- net at JP1.1 (A): now also MK1.5 (DOUT); no longer MK1.6 (VDD)
- net SDA1: now reaches U2.K17 (IO_EA_B2)
- net SDA1: now also R42.2, U11.B2 (SDA)
- net K8 renamed K5
- net power_supply/PG renamed SCL1
- net SCL1: now also R41.2, U11.A2 (SCL)
- no-connect marks 124 -> 122
Other:
- sheet power_supply ports: added none; removed PG
- note added: "1V1 2V5 3V3"
- note added: "Fiducial,Mechanical and mounting"
- note removed: "1V 2V5 3V3"
- note removed: "Mechanical mounting"
- moved on the sheet: JP1, MK1, R19, R20, TP1, TP2, TP3, TP4, U10

Commit message: start to switch to stm32
Parts:
- D15, D16: MPN PTVS5V0Z1USK -> PTVS5V0Z1USKYL
- FID1, FID2, FID3, FID4, FID5, FID6, J1, J4, TP5, TP6: MPN (none) -> DNP
- J3: MPN (none) -> 5024302030
- JP1: footprint Jumper:SolderJumper-2_P1.3mm_Open_RoundedPad1.0x1.5mm -> ProjectLibrary:Jumper_open
- MK1: MPN (none) -> CMM-4737DT-26386-TR
- N1: MPN (none) -> DNP; now not fitted
- P1: MPN (none) -> 1054440011
- TH1: value PTSLR06038V075 -> BSMD0603-075-6V
- TP1, TP2, TP3, TP4: MPN (none) -> DNP; now not fitted; now left out of the parts list
- U10: MPN (none) -> TMP110D
- U11: MPN (none) -> MMC5633NJL
- U5: MPN (none) -> USB3740B-AI2-TR
- U9: MPN (none) -> ISM330DHCXTR
Connections:
- net CC_CFG_CTRL_RECFG: now reaches U1.41 (GPIO27_ADC1)
- net CC_CFG_CTRL_RECFG: now also U2.V5 (IO_SA_B0)
- no-connect marks 122 -> 120
Other:
- moved on the sheet: R23

Commit message: draft layout
Parts:
- removed C55, C58: 100n, Capacitor_SMD:C_0402_1005Metric, symbol Device:C
- removed C56, C59, C60, C61, C62: 10n, Capacitor_SMD:C_0201_0603Metric, symbol Device:C
- removed C57: 1u, Capacitor_SMD:C_0402_1005Metric, symbol Device:C
- removed C6: 4u7, Capacitor_SMD:C_0402_1005Metric, symbol Device:C
- removed C7, C8: 15p, Capacitor_SMD:C_0402_1005Metric, symbol Device:C
- removed J1: Conn_02x02_Odd_Even, Connector_PinHeader_1.00mm:PinHeader_2x02_P1.00mm_Horizontal, symbol Connector_Generic:Conn_02x02_Odd_Even
- removed J3: 5024302030, Connector_Molex:Molex_SlimStack_502430-2010_2x10_P0.40mm_Vertical, symbol Connector_Generic:Conn_02x10_Odd_Even
- removed R1: 5K1, Resistor_SMD:R_0201_0603Metric, symbol Device:R_US
- removed TP5, TP6: TestPoint_Small, TestPoint:TestPoint_Pad_D1.0mm, symbol Connector:TestPoint_Small
- removed U1: RP2350A, RP2350_60QFN_minimal:RP2350-QFN-60-1EP_7x7_P0.4mm_EP3.4x3.4mm_ThermalVias, symbol MCU_RaspberryPi_RP2350:RP2350_60QFN
- removed Y2: ABM8-272-T3, Crystal:Crystal_SMD_3225-4Pin_3.2x2.5mm, symbol Device:Crystal_GND24
- added C118, C125: 100n, Capacitor_SMD:C_0402_1005Metric, symbol Device:C
- added C48, C49, C50, C51: 10n, Capacitor_SMD:C_0201_0603Metric, symbol Device:C
- added Q1: CSD25480F3, Package_DFN_QFN:Texas_PicoStar_DFN-3_0.69x0.60mm, symbol Transistor_FET:CSD25480F3
- added R45, R46: 0R, Resistor_SMD:R_0201_0603Metric, symbol Device:R_US
- added R47, R48, R49, R52: 5K1, Resistor_SMD:R_0201_0603Metric, symbol Device:R_US
- added R51: 1K5, Resistor_SMD:R_0201_0603Metric, symbol Device:R_US
- added SW1, SW2: KXT 331 LHS, Button_Switch_SMD:SW_SPST_CK_KXT3, symbol Switch:SW_Push
- added TP5, TP6, TP7, TP8: TestPoint, TestPoint:TestPoint_Pad_D1.0mm, symbol Connector:TestPoint
- added U1: TXS0202YZPR, Package_BGA:Texas_DSBGA-8_0.9x1.9mm_Layout2x4_P0.5mm, symbol TPSM8228222SILR:TXS0202YZPR
- added U12: STM32L422RBIx, Package_BGA:UFBGA-64_5x5mm_Layout8x8_P0.5mm, symbol MCU_ST_STM32L4:STM32L422RBIx
- C54: value 1u -> 10n; footprint Capacitor_SMD:C_0402_1005Metric -> Capacitor_SMD:C_0201_0603Metric
- C80: value 10n -> 100n; footprint Capacitor_SMD:C_0201_0603Metric -> Capacitor_SMD:C_0402_1005Metric
- C81: value 1u -> 100n
- R3: value 33R -> 5K1; footprint Resistor_SMD:R_0402_1005Metric -> Resistor_SMD:R_0201_0603Metric
- R38, R39: value 0R -> 5K1
Connections:
- net RUN is gone; now on net +2V5: R17.2
- net +1V1: no longer C54.1
- net +2V5: now also R3.1, C118.1, C125.1, C48.1, C49.1, C50.1, C51.1, R48.1, R49.1, U1.C1 (VCCA), U1.C2 (OE), U12.B2 (VBAT), U12.D2 (VDD), U12.E4 (VDD), U12.E6 (VDD), U12.H1 (VDDA); no longer R17.1, R38.1, R39.1
- net +3V3: now also C54.1, Q1.2 (S), U1.B2 (VCCB), U12.E5 (VDDUSB); no longer R3.2
- net CFG_MD2/IO_WA_A1: now also R39.1, U12.A4 (PB4); no longer R38.2
- net CFG_MD3/IO_WA_B1: now also R52.1, U12.A3 (PB9); no longer R39.2
- net FLASH_CLK: now also U2.N4 (IO_WA_B8/SPI_CLK), U12.G3 (PA3)
- net FLASH_S0: now also U2.P2 (IO_WA_B7/SPI_D0), U12.G5 (PB1)
- net FLASH_S1: now also U2.P1 (IO_WA_A7/SPI_D1), U12.F5 (PB0)
- net FLASH_S2: now also U2.R2 (IO_WA_B6/SPI_D2), U12.H4 (PA7)
- net FLASH_S3: now also U2.R1 (IO_WA_A6/SPI_D3), U12.G4 (PA6)
- net GND: now also R38.2, R39.2, C118.2, C125.2, C48.2, C49.2, C50.2, C51.2, R47.2, R52.2, SW1.1, SW2.1, U1.B1 (GND), U12.C2 (VSS), U12.D4 (VSS), U12.D5 (VSS), U12.D6 (VSS), U12.F1 (VSSA); no longer U2.R5 (CFG_MD0/IO_WA_A0), U2.T5 (CFG_MD1/IO_WA_B0)
- net RX0: now also U12.G7 (PB10); no longer U2.C18 (IO_EB_A4)
- net TX0: now also U12.H7 (PB11)
- net USB_DN: now also U12.C8 (PA11)
- net USB_DP: now also U12.B8 (PA12)
- net ~{FLASH_CS}: now also U2.N3 (IO_WA_A8/~{SPI_CS}), U12.F3 (PA2)
- net ~{RST}: now also TP7.1, U12.E1 (NRST); no longer R4.2, U2.T15 (~{RESET})
- net VBUS_UNPROTECTED: now reaches P1.A4 (VBUS), P1.A9 (VBUS), P1.B4 (VBUS), P1.B9 (VBUS), TH1.2
- net at P1.A5 (CC): now also R47.1
- net MCU_SCL: now reaches U2.G1 (IO_WC_A0)
- net MCU_SCL: now also R48.2, U12.G8 (PB13)
- net MCU_SDA: now reaches U2.G2 (IO_WC_B0)
- net MCU_SDA: now also R49.2, U12.F8 (PB14)
- net FPGA_USB_DN: now reaches U5.1 (DM_1)
- net FPGA_USB_DN: now also U1.A2 (BD-)
- net FPGA_USB_DP: now reaches U5.2 (DP_1)
- net FPGA_USB_DP: now also U1.A1 (BD+)
- net 2V5_FPGA_USB_DP: now reaches U2.U10 (IO_SA_A8)
- net 2V5_FPGA_USB_DP: now also R51.2, U1.D2 (AD-)
- net 2V5_FPGA_USB_DN: now reaches U2.V10 (IO_SA_B8)
- net 2V5_FPGA_USB_DN: now also U1.D1 (AD+)
- net USB_PU: now reaches U2.V8 (IO_SA_B5)
- net USB_PU: now also R46.1, U12.H8 (PB12)
- net CC_CFG_CTRL_CLK: no longer names the net of U2.B2 (IO_WC_B8)
- net CC_CFG_CTRL_EN: no longer names the net of U2.B1 (IO_WC_A8)
- net CC_CFG_CTRL_EN: no longer R23.1
- net CC_CFG_CTRL_RECFG: no longer names the net of U2.V5 (IO_SA_B0)
- net CC_CFG_CTRL_VALID: no longer names the net of U2.D2 (IO_WC_B5)
- net GPIO23_GPOUT1 renamed CLOCK_SYS
- net CLOCK_SYS: now also R45.1
- net HSTX_0_N: no longer names the net of U2.L2 (IO_WB_B3)
- net HSTX_0_P: no longer names the net of U2.L1 (IO_WB_A3)
- net HSTX_1_N: no longer names the net of U2.H2 (IO_WB_B7)
- net HSTX_1_P: no longer names the net of U2.H1 (IO_WB_A7)
- net HSTX_2_N: no longer names the net of U2.K2 (IO_WB_B5)
- net HSTX_2_P: no longer names the net of U2.K1 (IO_WB_A5)
- net HSTX_3_N: no longer names the net of U2.N2 (IO_WB_B0)
- net HSTX_3_P: no longer names the net of U2.N1 (IO_WB_A0)
- net RX1: no longer names the net of U2.C17 (IO_EB_B4)
- net TCK renamed FPGA_TCK
- net FPGA_TCK: now also U12.A1 (PC14)
- net TDI renamed FPGA_TDI
- net FPGA_TDI: now also U12.C1 (PH0)
- net TDO renamed FPGA_TDO
- net FPGA_TDO: now also U12.D1 (PH1)
- net TMS renamed FPGA_TMS
- net FPGA_TMS: now also U12.B1 (PC15)
- new net: Q1.1 (G), R17.1, R46.2
- new net: Q1.3 (D), R51.1
- new net BOOT0: R3.2, SW1.2, TP8.1, U12.B4 (PH3)
- new net CFG_MD0/IO_WA_A0: R23.1, U12.A6 (PA15), U2.R5 (CFG_MD0/IO_WA_A0)
- new net CFG_MD1/IO_WA_B0: R38.1, U12.A5 (PB3), U2.T5 (CFG_MD1/IO_WA_B0)
- new net RCC_MCO: R45.2, U12.D7 (PA8)
- new net SWCLK: TP6.1, U12.A7 (PA14)
- new net SWDIO: TP5.1, U12.A8 (PA13)
- new net ~{FPGA_RST}: R4.2, SW2.2, U12.H2 (PA1), U2.T15 (~{RESET})
- no-connect marks 120 -> 144
Other:
- note removed: "CX1 = 2(CL - Cstray) CL = 10pF Cstray = 2pF CX1 = 2(10-2) = 16pF"
- moved on the sheet: C46, C47, C52, C65, C66, C67, C68, C69, C70, C71, C72, C73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
