File: Expansion_Card_Retrofit.kicad_pcb (KiCad board)
At the start: 8 copper layers, 24 x 27.3 mm, 198 parts, among them J1 Conn_02x02_Odd_Even, J3 5024302030, J4 Conn_02x02_Odd_Even, P1 1054440011, U1 RP2350A, U10 TMP110D, U11 MMC5633NJL, U2 CCGM1A1, U3 TVS0500DRV, U4 W25Q16JLUXIG TR, U5 USB3740B-AI2, U6 TPS7A2033PDQNR, U7 TPSM82822SILR, U8 TPSM82822SILR, U9 ISM330DHCX, Y1 S3A2505-100.000-L-X1-R, Y2 ABM8-272-T3

Commit message: draft layout
Parts:
- removed C55, C58: 100n, Capacitor_SMD:C_0402_1005Metric
- removed C56, C59, C60, C61, C62: 10n, Capacitor_SMD:C_0201_0603Metric
- removed C57: 1u, Capacitor_SMD:C_0402_1005Metric
- removed C6: 4u7, Capacitor_SMD:C_0402_1005Metric
- removed C7, C8: 15p, Capacitor_SMD:C_0402_1005Metric
- removed J1: Conn_02x02_Odd_Even, Connector_PinHeader_1.00mm:PinHeader_2x02_P1.00mm_Horizontal
- removed J3: 5024302030, Connector_Molex:Molex_SlimStack_502430-2010_2x10_P0.40mm_Vertical
- removed R1: 5K1, Resistor_SMD:R_0201_0603Metric
- removed Y2: ABM8-272-T3, Crystal:Crystal_SMD_3225-4Pin_3.2x2.5mm
- added C118: 100n, Capacitor_SMD:C_0402_1005Metric, B.Cu at (143.2, 135.4)
- added C125: 100n, Capacitor_SMD:C_0402_1005Metric, B.Cu at (150.7, 130.5)
- added C48: 10n, Capacitor_SMD:C_0201_0603Metric, B.Cu at (149.5, 133.6)
- added C49: 10n, Capacitor_SMD:C_0201_0603Metric, B.Cu at (146.9, 132.7)
- added C50: 10n, Capacitor_SMD:C_0201_0603Metric, B.Cu at (148.7, 133.2)
- added C51: 10n, Capacitor_SMD:C_0201_0603Metric, B.Cu at (151.1, 131.7)
- added Q1: CSD25480F3, Package_DFN_QFN:Texas_PicoStar_DFN-3_0.69x0.60mm, B.Cu at (141.7, 136.9)
- added R45: 0R, Resistor_SMD:R_0201_0603Metric, B.Cu at (146.6, 133.4)
- added R46: 0R, Resistor_SMD:R_0201_0603Metric, B.Cu at (142.8, 137.2)
- added R47: 5K1, Resistor_SMD:R_0201_0603Metric, F.Cu at (139.2, 131.8)
- added R48: 5K1, Resistor_SMD:R_0201_0603Metric, B.Cu at (155.6, 146.8)
- added R49: 5K1, Resistor_SMD:R_0201_0603Metric, B.Cu at (155.6, 148.6)
- added R51: 1K5, Resistor_SMD:R_0201_0603Metric, B.Cu at (142.8, 136.5)
- added R52: 5K1, Resistor_SMD:R_0201_0603Metric, B.Cu at (147.6, 136.6)
- added SW1: KXT 331 LHS, Button_Switch_SMD:SW_SPST_CK_KXT3, F.Cu at (130.3, 152.4)
- added SW2: KXT 331 LHS, Button_Switch_SMD:SW_SPST_CK_KXT3, B.Cu at (130.3, 152.4)
- added TP7: TestPoint, TestPoint:TestPoint_Pad_D1.0mm, B.Cu at (151.0, 133.4)
- added TP8: TestPoint, TestPoint:TestPoint_Pad_D1.0mm, B.Cu at (148.6, 135.2)
- added U12: STM32L422RBIx, Package_BGA:UFBGA-64_5x5mm_Layout8x8_P0.5mm, F.Cu at (148.2, 133.2)
- C46, C47, R12, R34, U4: moved to F.Cu
- C54: value 1u -> 10n; footprint Capacitor_SMD:C_0402_1005Metric -> Capacitor_SMD:C_0201_0603Metric; moved to B.Cu
- C78, C79, R23, U3: moved to B.Cu
- C80: value 10n -> 100n; footprint Capacitor_SMD:C_0201_0603Metric -> Capacitor_SMD:C_0402_1005Metric; moved to B.Cu
- C81: value 1u -> 100n; moved to B.Cu
- R3: value 33R -> 5K1; footprint Resistor_SMD:R_0402_1005Metric -> Resistor_SMD:R_0201_0603Metric; moved to F.Cu
- R38, R39: value 0R -> 5K1
- TH1: value PTSLR06038V075 -> BSMD0603-075-6V; moved to B.Cu
- TP5, TP6: value TestPoint_Small -> TestPoint
- U1: value RP2350A -> TXS0202YZPR; footprint RP2350_60QFN_minimal:RP2350-QFN-60-1EP_7x7_P0.4mm_EP3.4x3.4mm_ThermalVias -> Package_BGA:Texas_DSBGA-8_0.9x1.9mm_Layout2x4_P0.5mm; moved to F.Cu
- moved FID6 23.9 mm to (151.2, 137.6)
- moved R12 20.3 mm to (149.9, 144.2), turned to 180 degrees
- moved R23 17.6 mm to (145.5, 136.6), turned to -90 degrees
- moved R17 16.3 mm to (141.5, 138.2), turned to -90 degrees
- moved C47 16.1 mm to (149.5, 138.4), turned to 0 degrees
- moved C46 15.7 mm to (149.4, 139.2), turned to 0 degrees
- moved U4 15.0 mm to (150.0, 141.7), turned to 90 degrees
- moved R3 14.2 mm to (130.4, 149.9), turned to 0 degrees
- moved U3 12.4 mm to (137.7, 135.3), turned to 90 degrees
- moved TP6 8.43 mm to (144.6, 131.7)
- moved TH1 8.38 mm to (137.9, 133.1), turned to 0 degrees
- moved C79 7.15 mm to (144.7, 139.1), turned to 180 degrees
- moved TP5 6.68 mm to (145.4, 134.9)
- moved C78 4.92 mm to (148.2, 139.7)
- moved R38 4.78 mm to (146.2, 136.6), turned to -90 degrees
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Connections:
- net Net-(P1-VBUS-PadA4) renamed /VBUS_UNPROTECTED
- C54 pad 1: +1V1 -> +3V3
- R17 pad 1: +2V5 -> Net-(Q1-G)
- R17 pad 2: /RUN -> +2V5
- R23 pad 1: /CC_CFG_CTRL_EN -> /CFG_MD0/IO_WA_A0
- R3 pad 1: Net-(U1-VREG_AVDD) -> +2V5
- R3 pad 2: +3V3 -> /BOOT0
- R38 pad 1: +2V5 -> /CFG_MD1/IO_WA_B0
- R38 pad 2: /CFG_MD2/IO_WA_A1 -> GND
- R39 pad 1: +2V5 -> /CFG_MD2/IO_WA_A1
- R39 pad 2: /CFG_MD3/IO_WA_B1 -> GND
- R4 pad 2: /~{RST} -> /~{FPGA_RST}
- TP5 pad 1: Net-(U1-SWCLK) -> /SWDIO
- TP6 pad 1: Net-(U1-SWD) -> /SWCLK
- U2 pad B1: /CC_CFG_CTRL_EN -> unconnected-(U2F-IO_WC_A8-PadB1)
- U2 pad B2: /CC_CFG_CTRL_CLK -> unconnected-(U2F-IO_WC_B8-PadB2)
- U2 pad C17: /RX1 -> unconnected-(U2D-IO_EB_B4-PadC17)
- U2 pad C18: /RX0 -> unconnected-(U2D-IO_EB_A4-PadC18)
- U2 pad D2: /CC_CFG_CTRL_VALID -> unconnected-(U2F-IO_WC_B5-PadD2)
- U2 pad G1: unconnected-(U2F-IO_WC_A0-PadG1) -> /MCU_SCL
- U2 pad G2: unconnected-(U2F-IO_WC_B0-PadG2) -> /MCU_SDA
- U2 pad H1: /HSTX_1_P -> unconnected-(U2F-IO_WB_A7-PadH1)
- U2 pad H2: /HSTX_1_N -> unconnected-(U2F-IO_WB_B7-PadH2)
- U2 pad K1: /HSTX_2_P -> unconnected-(U2F-IO_WB_A5-PadK1)
- U2 pad K2: /HSTX_2_N -> unconnected-(U2F-IO_WB_B5-PadK2)
- U2 pad L1: /HSTX_0_P -> unconnected-(U2F-IO_WB_A3-PadL1)
- U2 pad L2: /HSTX_0_N -> unconnected-(U2F-IO_WB_B3-PadL2)
- U2 pad N1: /HSTX_3_P -> unconnected-(U2F-IO_WB_A0-PadN1)
- U2 pad N2: /HSTX_3_N -> unconnected-(U2F-IO_WB_B0-PadN2)
- U2 pad N3: Net-(J3-Pin_11) -> /~{FLASH_CS}
- U2 pad N4: Net-(J3-Pin_13) -> /FLASH_CLK
- U2 pad P1: Net-(J3-Pin_5) -> /FLASH_S1
- U2 pad P12: /GPIO23_GPOUT1 -> /CLOCK_SYS
- U2 pad P2: Net-(J3-Pin_3) -> /FLASH_S0
- U2 pad R1: Net-(J3-Pin_9) -> /FLASH_S3
- U2 pad R2: Net-(J3-Pin_7) -> /FLASH_S2
- U2 pad R3: /TCK -> /FPGA_TCK
- U2 pad R5: GND -> /CFG_MD0/IO_WA_A0
- U2 pad T15: /~{RST} -> /~{FPGA_RST}
- U2 pad T2: /TDI -> /FPGA_TDI
- U2 pad T3: /TMS -> /FPGA_TMS
- U2 pad T5: GND -> /CFG_MD1/IO_WA_B0
- U2 pad U10: unconnected-(U2E-IO_SA_A8-PadU10) -> /2V5_FPGA_USB_DP
- U2 pad U2: /TDO -> /FPGA_TDO
- U2 pad V10: unconnected-(U2E-IO_SA_B8-PadV10) -> /2V5_FPGA_USB_DN
- U2 pad V5: /CC_CFG_CTRL_RECFG -> unconnected-(U2E-IO_SA_B0-PadV5)
- U2 pad V8: unconnected-(U2E-IO_SA_B5-PadV8) -> /USB_PU
- U5 pad 1: unconnected-(U5-DM_1-Pad1) -> /FPGA_USB_DN
- U5 pad 2: unconnected-(U5-DP_1-Pad2) -> /FPGA_USB_DP
Routing:
- net /~{RST}: track 69.5 -> 1.22 mm, vias 3 -> 1
- net /~{FPGA_RST}: track 0.00 -> 37.8 mm, vias 0 -> 3
- net /~{FLASH_CS}: track 40.9 -> 6.49 mm, vias 2 -> 3
- net /RUN: track 32.6 -> 0.00 mm, vias 1 -> 0
- net /TX1: track 30.5 -> 0.00 mm, vias 2 -> 0
- net /CC_CFG_CTRL_VALID: track 27.6 -> 0.00 mm, vias 2 -> 0
- net GND: track 139.0 -> 112.1 mm, vias 128 -> 133
- net Net-(U2B-IO_WA_B2/CFG_DONE): track 27.1 -> 0.63 mm, vias 2 -> 1
- net /RX1: track 25.8 -> 0.00 mm, vias 2 -> 0
- net +2V5: track 87.5 -> 62.0 mm, vias 74 -> 76
- net /HSTX_1_N: track 24.7 -> 0.00 mm, vias 2 -> 0
- net /TX0: track 25.2 -> 0.65 mm, vias 2 -> 1
- net /RX0: track 24.3 -> 0.00 mm, vias 2 -> 1
- net /HSTX_1_P: track 23.7 -> 0.00 mm, vias 2 -> 0
- net /HSTX_0_N: track 23.4 -> 0.00 mm, vias 3 -> 0
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- removed copper zone on F.Cu, net +3V3
- removed copper zone on In4.Cu, net VBUS
- removed copper zone on In5.Cu, net VBUS
Other:
- board text added: "BOOT0"
- board text added: "~{F_RST}"

Commit message: testbench done
Parts:
- removed U3: TVS0500DRV, Package_SON:WSON-6-1EP_2x2mm_P0.65mm_EP1x1.6mm
- added C119: 1u, Capacitor_SMD:C_0402_1005Metric, B.Cu at (149.6, 138.5)
- added D17: PTVS5V0Z1USK, Diode_SMD:Nexperia_DSN1608-2_1.6x0.8mm, B.Cu at (140.8, 131.7)
- added R50: 5K1, Resistor_SMD:R_0201_0603Metric, B.Cu at (151.6, 131.7)
- added R53: 5K1, Resistor_SMD:R_0201_0603Metric, B.Cu at (130.5, 149.2)
- R12: moved to B.Cu
- moved R49 9.49 mm to (146.2, 147.6), turned to 0 degrees
- moved R48 8.32 mm to (147.3, 147.3), turned to -90 degrees
- moved FID1 2.61 mm to (145.6, 144.6)
- moved TP7 2.16 mm to (150.1, 135.3)
- moved R12 0.88 mm to (149.0, 144.1), turned to 90 degrees
- moved TP8 0.62 mm to (148.0, 134.9)
- moved TP5 0.59 mm to (146.0, 134.9)
- moved FID4 0.38 mm to (130.4, 137.3)
- moved C51 0.19 mm to (150.9, 131.7)
- moved C81 0.18 mm to (143.4, 134.5)
Connections:
- U2 pad D17: /TX1 -> /RX0
Routing:
- net /BOOT0: track 1.57 -> 32.8 mm, vias 1 -> 2
- net /TX0: track 0.65 -> 29.1 mm, vias 1 -> 2
- net /RX0: track 0.00 -> 28.4 mm, vias 1 -> 2
- net /MCU_SDA: track 0.58 -> 23.9 mm, vias 1 -> 3
- net /MCU_SCL: track 1.08 -> 22.7 mm, vias 1 -> 3
- net /~{FLASH_CS}: track 6.49 -> 27.8 mm
- net Net-(U2B-IO_WA_B2/CFG_DONE): track 0.63 -> 17.1 mm, vias 1 -> 2
- net /VBUS_UNPROTECTED: track 16.0 -> 2.50 mm
- net /FLASH_S1: track 8.81 -> 21.8 mm, vias 1 -> 2
- net /FLASH_S2: track 9.97 -> 22.7 mm, vias 1 -> 2
- net /power_supply/PG_2V5: track 1.17 -> 12.9 mm, vias 1 -> 2
- net /USB_PU: track 3.42 -> 14.0 mm
- net /FLASH_CLK: track 7.73 -> 17.6 mm
- net /FPGA_TDI: track 0.59 -> 9.26 mm, vias 1 -> 2
- net /~{RST}: track 1.22 -> 9.75 mm, vias 1 -> 2
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- added copper zone on In4.Cu, net +3V3
- added copper zone on B.Cu, net /VBUS_UNPROTECTED
Other:
- board text added: "+3V3"
- board text added: "MCU"

Commit message: fixed diff pair
Parts:
- U12: value STM32L422RBIx -> STM32L422RBI6
- moved C1 0.74 mm to (133.8, 130.7), turned to -90 degrees
- moved D17 0.10 mm to (140.8, 131.8)
- moved TP6 0.09 mm to (144.7, 131.8)
Routing:
- net /RX1_P: track 17.5 -> 12.3 mm
- net GND: track 112.0 -> 109.3 mm, vias 130 -> 133
- net /RX2_N: track 26.1 -> 23.5 mm
- net /RX2_P: track 25.4 -> 23.4 mm
- net Net-(P1-SHIELD): track 17.2 -> 15.7 mm
- net +2V5: track 63.1 -> 64.5 mm
- net /TX2_N: track 28.3 -> 29.3 mm
- net /RX1_N: track 14.5 -> 13.8 mm
- net /FPGA_USB_DN: track 9.42 -> 8.68 mm
- net /FLASH_S3: track 14.4 -> 14.9 mm
- net /FLASH_S1: track 21.8 -> 22.3 mm
Other:
- board text added: "B0"
- board text added: "SWDIO"
- board text added: "~{RST}"
- board text removed: "SWD"
